File: ai03-pcb-test-time.sch (KiCad schematic (older format))
At the start: 24 parts, among them SW1 SW_Push, U1 ATmega32U4-AU, Y1 16MHz

Commit message: Schematic fixed
Connections:
- net D+: now also USB1.3 (D+); no longer USB1.4 (D-)
- net D-: now also USB1.4 (D-); no longer USB1.5 (VBUS)
- net GND: now also USB1.1 (GND)
- net VCC: now also USB1.5 (VBUS); no longer USB1.6 (SHIELD)
Other:
- moved on the sheet: F1
Changed lines of the file:
@@
 L Device:Polyfuse_Small F1
 U 1 1 5D229526
-P 2350 850
-F 0 "F1" V 2145 850 50  0000 C CNN
-F 1 "Polyfuse_Small" V 2236 850 50  0000 C CNN
-F 2 "Inductor_SMD:L_1206_3216Metric" H 2400 650 50  0001 L CNN
-F 3 "~" H 2350 850 50  0001 C CNN
-	1    2350 850
+P 2350 950
+F 0 "F1" V 2145 950 50  0000 C CNN
+F 1 "Polyfuse_Small" V 2236 950 50  0000 C CNN
+F 2 "Inductor_SMD:L_1206_3216Metric" H 2400 750 50  0001 L CNN
+F 3 "~" H 2350 950 50  0001 C CNN
+	1    2350 950
 	0    1    1    0
 $EndComp
@@
 L power:VCC #PWR0111
 U 1 1 5D2295D3
-P 1800 850
-F 0 "#PWR0111" H 1800 700 50  0001 C CNN
-F 1 "VCC" H 1817 1023 50  0000 C CNN
-F 2 "" H 1800 850 50  0001 C CNN
-F 3 "" H 1800 850 50  0001 C CNN
-	1    1800 850
+P 1800 950
+F 0 "#PWR0111" H 1800 800 50  0001 C CNN
+F 1 "VCC" H 1817 1123 50  0000 C CNN
+F 2 "" H 1800 950 50  0001 C CNN
+F 3 "" H 1800 950 50  0001 C CNN
+	1    1800 950
 	1    0    0    -1
 $EndComp
@@
 L power:+5V #PWR0112
 U 1 1 5D229841
-P 2950 850
-F 0 "#PWR0112" H 2950 700 50  0001 C CNN
-F 1 "+5V" H 2965 1023 50  0000 C CNN
-F 2 "" H 2950 850 50  0001 C CNN
-F 3 "" H 2950 850 50  0001 C CNN
-	1    2950 850
+P 2950 950
+F 0 "#PWR0112" H 2950 800 50  0001 C CNN
+F 1 "+5V" H 2965 1123 50  0000 C CNN
+F 2 "" H 2950 950 50  0001 C CNN
+F 3 "" H 2950 950 50  0001 C CNN
+	1    2950 950
 	1    0    0    -1
 $EndComp
 Wire Wire Line
-	2950 850  2450 850
+	2950 950  2450 950
 Wire Wire Line
-	2250 850  1800 850
+	2250 950  1800 950
 Wire Wire Line
-	1800 850  1350 850
-Connection ~ 1800 850
-Text GLabel 1350 950  2    50   Input ~ 0
+	1800 950  1350 950
+Connection ~ 1800 950
+Text GLabel 1350 1050 2    50   Input ~ 0
 D-
-Text GLabel 1350 1050 2    50   Input ~ 0
+Text GLabel 1350 1150 2    50   Input ~ 0
 D+
 $Comp
@@
 Text GLabel 2200 2950 1    50   Input ~ 0
 COL1
+$Comp
+L power:GND #PWR?
+U 1 1 5D240C66
+P 1500 1350
+F 0 "#PWR?" H 1500 1100 50  0001 C CNN
+F 1 "GND" H 1505 1177 50  0000 C CNN
+F 2 "" H 1500 1350 50  0001 C CNN
+F 3 "" H 1500 1350 50  0001 C CNN
+	1    1500 1350
+	1    0    0    -1
+$EndComp
+Wire Wire Line
+	1500 1350 1350 1350
 $EndSCHEMATC

Commit message: Fixed schematic again
Parts:
- C3, C4: value C_Small -> 22pF
- F1: value Polyfuse_Small -> 500mA; footprint Inductor_SMD:L_1206_3216Metric -> Fuse:Fuse_1206_3216Metric
Changed lines of the file:
@@
 P 3870 2400
 F 0 "C3" V 3641 2400 50  0000 C CNN
-F 1 "C_Small" V 3732 2400 50  0000 C CNN
+F 1 "22pF" V 3732 2400 50  0000 C CNN
 F 2 "Capacitor_SMD:C_0805_2012Metric" H 3870 2400 50  0001 C CNN
 F 3 "~" H 3870 2400 50  0001 C CNN
@@
 P 3870 2920
 F 0 "C4" V 3641 2920 50  0000 C CNN
-F 1 "C_Small" V 3732 2920 50  0000 C CNN
+F 1 "22pF" V 3732 2920 50  0000 C CNN
 F 2 "Capacitor_SMD:C_0805_2012Metric" H 3870 2920 50  0001 C CNN
 F 3 "~" H 3870 2920 50  0001 C CNN
@@
 P 2350 950
 F 0 "F1" V 2145 950 50  0000 C CNN
-F 1 "Polyfuse_Small" V 2236 950 50  0000 C CNN
-F 2 "Inductor_SMD:L_1206_3216Metric" H 2400 750 50  0001 L CNN
+F 1 "500mA" V 2236 950 50  0000 C CNN
+F 2 "Fuse:Fuse_1206_3216Metric" H 2400 750 50  0001 L CNN
 F 3 "~" H 2350 950 50  0001 C CNN
 	1    2350 950
@@
 COL1
 $Comp
-L power:GND #PWR?
+L power:GND #PWR0113
 U 1 1 5D240C66
 P 1500 1350
-F 0 "#PWR?" H 1500 1100 50  0001 C CNN
+F 0 "#PWR0113" H 1500 1100 50  0001 C CNN
 F 1 "GND" H 1505 1177 50  0000 C CNN
 F 2 "" H 1500 1350 50  0001 C CNN
