File: ai03-pcb-test-time.kicad_pcb (KiCad board)
At the start: 2 copper layers, 24 parts, among them SW1 SW_Push, U1 ATmega32U4-AU, Y1 16MHz

Commit message: Schleep schoon
Parts:
- C3, C4: value C_Small -> 22pF
- F1: value Polyfuse_Small -> 500mA; footprint Inductor_SMD:L_1206_3216Metric -> Fuse:Fuse_1206_3216Metric
- moved C2 101.2 mm to (67.9, 22.5), turned to 0 degrees
- moved C7 94.0 mm to (81.3, 36.4)
- moved C1 86.1 mm to (67.9, 24.5), turned to 0 degrees
- moved C5 76.5 mm to (91.0, 43.8), turned to 0 degrees
- moved Y1 73.2 mm to (73.1, 28.4), turned to 0 degrees
- moved C4 70.5 mm to (95.6, 48.0), turned to 0 degrees
- moved C3 64.3 mm to (91.0, 45.7), turned to 0 degrees
- moved D3 60.6 mm to (123.8, 81.0)
- moved USB1 35.6 mm to (33.3, 61.1)
- moved R1 34.3 mm to (31.0, 70.6), turned to 90 degrees
- moved R2 34.3 mm to (33.3, 70.6)
- moved D1 33.7 mm to (104.8, 81.0)
- moved D4 33.7 mm to (123.8, 100.0)
- moved MX1 33.7 mm to (96.8, 81.0)
- moved MX2 33.7 mm to (96.8, 100.0)
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Connections:
- USB1 pad 1: Net-(USB1-Pad1) -> GND
- USB1 pad 3: Net-(USB1-Pad3) -> D+
- USB1 pad 4: D+ -> D-
- USB1 pad 5: D- -> VCC
- USB1 pad 6: VCC -> Net-(USB1-Pad6)

Commit message: Schleep for real
Parts:
- moved C7 72.8 mm to (42.1, 97.6)
- moved C5 72.4 mm to (35.7, 90.5), turned to 270 degrees
- moved C2 63.7 mm to (44.5, 81.8)
- moved C1 61.8 mm to (54.8, 84.9), turned to 90 degrees
- moved C4 56.1 mm to (47.6, 77.0), turned to 270 degrees
- moved Y1 53.1 mm to (51.6, 77.0), turned to 180 degrees
- moved C3 47.3 mm to (55.6, 77.0), turned to 90 degrees
- moved USB1 15.2 mm to (31.8, 76.2)
- moved R1 13.5 mm to (31.8, 84.1)
- moved R2 13.5 mm to (34.1, 84.1)
- moved F1 11.3 mm to (29.4, 84.9)
- moved SW1 7.14 mm to (31.0, 94.5), turned to 270 degrees
- moved R3 3.55 mm to (42.1, 79.4)
- moved C6 2.25 mm to (38.1, 90.5)
